File: hardware/pico_dual_sided/pico_dual_sided.kicad_pcb (KiCad board)
At the start: 2 copper layers, 179.7 x 119.4 mm, 89 parts, among them IC1 REYAX_RYLR896, J1 Conn_01x04, SW1 SW_MEC_5E, SW10 SW_MEC_5E, SW11 SW_MEC_5E, SW12 SW_MEC_5E, SW13 SW_MEC_5E, SW14 SW_MEC_5E, SW15 SW_MEC_5E, SW16 SW_MEC_5E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

Commit message: changes to hardware
Routing:
- net Net-(IC1-Pad6): track 129.2 -> 143.8 mm
- net Net-(IC1-Pad4): track 76.8 -> 84.1 mm
- net Net-(J1-Pad1): track 105.2 -> 111.4 mm, vias 2 -> 0
- net Net-(J1-Pad3): vias 0 -> 2
